Commit message: mass & inertia input but not done

File: franka_description/robots/panda_arm.xacro (robot description, xacro)
@@ -32,6 +32,7 @@
       <inertial>
         <origin xyz="0 0 0" rpy="0 0 0" />
-        <mass value="3.06" />
-        <inertia ixx="0.3" ixy="0.0" ixz="0.0" iyy="0.3" iyz="0.0" izz="0.3" />
+        <mass value="4.6165" />
+        <inertia ixx="1.5938" ixy="0.1074" ixz="0.0032
+            " iyy="1.5938" iyz="0.0014" izz="0.0212" />
       </inertial>
       <!-- end for simulation -->
@@ -51,6 +52,6 @@
       <inertial>
         <origin xyz="0 0 0" rpy="0 0 0" />
-        <mass value="2.34" />
-        <inertia ixx="0.3" ixy="0.0" ixz="0.0" iyy="0.3" iyz="0.0" izz="0.3" />
+        <mass value="4.4735" />
+        <inertia ixx="0.1036" ixy="-0.0053" ixz="0.0284" iyy="0.0078" iyz="-0.0035" izz="0.1568" />
       </inertial>
       <!-- end for simulation -->
@@ -81,6 +82,6 @@
       <inertial>
         <origin xyz="0 0 0" rpy="0 0 0" />
-        <mass value="2.36" />
-        <inertia ixx="0.3" ixy="0.0" ixz="0.0" iyy="0.3" iyz="0.0" izz="0.3" />
+        <mass value="2.6049" />
+        <inertia ixx="0.0874" ixy="0.0008" ixz="-0.0107" iyy="0.0895" iyz="0.0" izz="0.3" />
       </inertial>
       <!-- end for simulation -->
@@ -111,5 +112,5 @@
       <inertial>
         <origin xyz="0 0 0" rpy="0 0 0" />
-        <mass value="2.38" />
+        <mass value="2.5037" />
         <inertia ixx="0.3" ixy="0.0" ixz="0.0" iyy="0.3" iyz="0.0" izz="0.3" />
       </inertial>
@@ -141,5 +142,5 @@
       <inertial>
         <origin xyz="0 0 0" rpy="0 0 0" />
-        <mass value="2.43" />
+        <mass value="1.8632" />
         <inertia ixx="0.3" ixy="0.0" ixz="0.0" iyy="0.3" iyz="0.0" izz="0.3" />
       </inertial>
@@ -171,5 +172,5 @@
       <inertial>
         <origin xyz="0 0 0" rpy="0 0 0" />
-        <mass value="3.5" />
+        <mass value="1.3229" />
         <inertia ixx="0.3" ixy="0.0" ixz="0.0" iyy="0.3" iyz="0.0" izz="0.3" />
       </inertial>
@@ -201,5 +202,5 @@
       <inertial>
         <origin xyz="0 0 0" rpy="0 0 0" />
-        <mass value="1.47" />
+        <mass value="0.9699" />
         <inertia ixx="0.3" ixy="0.0" ixz="0.0" iyy="0.3" iyz="0.0" izz="0.3" />
       </inertial>
